File: pcb/blinkenbrain.kicad_sch (KiCad schematic)
At the start: 29 parts, among them Q1 BC847BS, Q2 NX6008NBKW, SW1 SC-01KP, U1 TPS613222ADBVR

Commit message: Initial revision D
- Parts optimized for JLCPCB production
- Awaiting on some digikey sourced parts to reach their warehouse. I
will then use these design files and either merge or update if changes
are needed.
Parts:
- removed Q2: NX6008NBKW, Package_TO_SOT_SMD:SOT-323_SC-70, symbol Transistor_FET:BS170F
- added U2: LMV321AIDCKR, Package_TO_SOT_SMD:SOT-353_SC-70-5, symbol Amplifier_Operational:LMV321
- BT1: LCSC (none) -> C5213768
- C1, C2, C3: LCSC (none) -> C516003
- C4, C5, C6: LCSC (none) -> C19702
- C7: LCSC (none) -> C59302
- D1: LCSC (none) -> C7129856
- L1: LCSC (none) -> C391305
- Q1: LCSC (none) -> C8653
- R1, R2, R9: footprint Resistor_SMD:R_0402_1005Metric -> Resistor_SMD:R_0603_1608Metric; LCSC (none) -> C2907015
- R3, R4, R8: LCSC (none) -> C2906872
- R5, R6: LCSC (none) -> C60491
- R7: value 470 -> 120; LCSC (none) -> C2906988
- RV1: LCSC (none) -> C719186
- SW1: value SC-01KP -> 2.54-1P TPGT; footprint open-ephys:DEALON_DIP_SPSTx01_SC-01KP_W7.62mm_P1.27mm -> Button_Switch_SMD:SW_DIP_SPSTx01_Slide_6.7x4.1mm_W8.61mm_P2.54mm_LowProfile; LCSC (none) -> C7421519
- U1: LCSC (none) -> C2071163
Connections:
- net +5V: now also U2.5 (V+); no longer R7.2
- net GND: now also R7.1, U2.2 (V-)
- net at Q1.3 (C2), R6.1: now also U2.1 (+)
- net at D1.2 (A): now also U2.4; no longer R7.1
- net at D1.1 (K): now also R7.2, U2.3 (-)
- net LED_{En}: no longer names the net of Q1.6 (C1), R1.2, R2.1, R5.2, TP4.1
Other:
- moved on the sheet: C2, C3, D1, R4, R7, TP1
